File: ESP32-Simple-Thermostat-PCB/ESP32-Simple-Thermostat-PCB_no-route.kicad_pcb (KiCad board)
At the start: 2 copper layers, 133 x 89.5 mm, 47 parts, among them J1 PINHD_1x18_Male, J2 Screw_Terminal_9_P3.50mm, J3 DS18B20, J4 3.2 lcd tft, K1 G5Q-1A, K2 G5Q-1A, K3 G5Q-1A, K4 G5Q-1A, K5 G5Q-1A, K6 G5Q-1A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

Commit message: modified:   ESP32-Simple-Thermostat-PCB/ESP32-Simple-Thermostat-PCB.kicad_pcb 	new file:   ESP32-Simple-Thermostat-PCB/ESP32-Simple-Thermostat-PCB_no-route-backups/ESP32-Simple-Thermostat-PCB_no-route-2025-11-18_112218.zip 	modified:   ESP32-Simple-Thermostat-PCB/ESP32-Simple-Thermostat-PCB_no-route.kicad_pcb 	new file:   ESP32-Simple-Thermostat-PCB/ESP32-Simple-Thermostat-PCB_no-route.kicad_prl 	deleted:    ESP32-Simple-Thermostat-PCB/_autosave-ESP32-Simple-Thermostat-PCB.kicad_pcb 	modified:   ESP32-Simple-Thermostat-PCB/jlcpcb/gerber/ESP32-Simple-Thermostat-PCB-CuBottom.gbr 	modified:   ESP32-Simple-Thermostat-PCB/jlcpcb/gerber/ESP32-Simple-Thermostat-PCB-CuTop.gbr 	modified:   ESP32-Simple-Thermostat-PCB/jlcpcb/gerber/ESP32-Simple-Thermostat-PCB-EdgeCuts.gbr 	modified:   ESP32-Simple-Thermostat-PCB/jlcpcb/gerber/ESP32-Simple-Thermostat-PCB-MaskBottom.gbr 	modified:   ESP32-Simple-Thermostat-PCB/jlcpcb/gerber/ESP32-Simple-Thermostat-PCB-MaskTop.gbr 	modified:   ESP32-Simple-Thermostat-PCB/jlcpcb/gerber/ESP32-Simple-Thermostat-PCB-NPTH-drl_map.pdf 	modified:   ESP32-Simple-Thermostat-PCB/jlcpcb/gerber/ESP32-Simple-Thermostat-PCB-NPTH.drl 	modified:   ESP32-Simple-Thermostat-PCB/jlcpcb/gerber/ESP32-Simple-Thermostat-PCB-PTH-drl_map.pdf 	modified:   ESP32-Simple-Thermostat-PCB/jlcpcb/gerber/ESP32-Simple-Thermostat-PCB-PTH.drl 	modified:   ESP32-Simple-Thermostat-PCB/jlcpcb/gerber/ESP32-Simple-Thermostat-PCB-SilkBottom.gbr 	modified:   ESP32-Simple-Thermostat-PCB/jlcpcb/gerber/ESP32-Simple-Thermostat-PCB-SilkTop.gbr 	modified:   ESP32-Simple-Thermostat-PCB/jlcpcb/production_files/BOM-ESP32-Simple-Thermostat-PCB.csv 	modified:   ESP32-Simple-Thermostat-PCB/jlcpcb/production_files/CPL-ESP32-Simple-Thermostat-PCB.csv 	modified:   ESP32-Simple-Thermostat-PCB/jlcpcb/production_files/GERBER-ESP32-Simple-Thermostat-PCB.zip 	modified:   ESP32-Simple-Thermostat-PCB/jlcpcb/project.db
Parts:
- removed H5, H6, H7, H8: MountingHole_M3_3.2mm_Pad, PCM_SL_Mechanical:MountingHole_3.2mm_Pad
- added ?: , , F.Cu at (67.1, 44.1)
- added ?: , , F.Cu at (67.1, 93.0)
- added ?: , , F.Cu at (150.2, 93.0)
- added ?: , , F.Cu at (150.2, 44.1)
